File: schema.kicad_sch (KiCad schematic)
At the start: 15 parts, among them J1 DC/DC Boost Input, J2 DC/DC Boost output, J3 Retroilluminazione, J4 RPM Out, Q1 2N2222, Q2 S9018, Q3 2N2222

Commit message: step 2
Parts:
- removed C2: 10nF, Capacitor_THT:C_Axial_L3.8mm_D2.6mm_P7.50mm_Horizontal, symbol Device:C
- removed Q2: S9018, Package_TO_SOT_THT:TO-92S, symbol Device:Q_NPN
- removed R4: 10K, Resistor_THT:R_Axial_DIN0204_L3.6mm_D1.6mm_P5.08mm_Horizontal, symbol Device:R_Small
- C1: value 10nF -> 150pF
- Q1, Q3: value 2N2222 -> S8050
- R1: value 830 -> 380
- R2: value 10K -> 1K
- R3: value 1K -> 680K
Connections:
- net +11.2V: now also J4.2 (Pin_2); no longer Q3.3 (C), R3.1
- net GND: now also Q3.1 (E), R3.1; no longer J4.1 (Pin_1)
- net at C1.1, R5.1: now also R2.2, R3.2
- new net: J4.1 (Pin_1), Q3.3 (C)
Other:
- moved on the sheet: C1, J4, Q3, R2, R5
